Commit message: feat: refactor the .urdf.xacro with apriltag for mini and remove useless *.urdf

File: tianbot_mini/urdf/tianbot_mini.urdf.xacro (robot description, xacro)
@@ -53,4 +53,46 @@
       </xacro:if>
     </xacro:if>
+      <link name="${namespace}${name}">
+      <inertial>
+        <mass value="0.001" />
+        <origin xyz="0 0 0" rpy="0 0 0" />
+        <inertia ixx="0.00001" ixy="0" ixz="0" iyy="0.00001" iyz="0" izz="0.00002" />
+      </inertial>
+      <collision>
+        <origin xyz="0 0 0" rpy="0 0 0" />
+        <geometry>
+          <box size="${mesh_size} ${mesh_size} 0.001" />
+        </geometry>
+      </collision>
+      <visual>
+        <origin xyz="0 0 0" rpy="0 0 0" />
+        <geometry>
+          <!-- use Python str to convert family name and to generate leading zeros -->
+          <mesh filename="package://tams_apriltags/meshes/tag${str(family).replace( 'h', '_' )}_${str(ID).zfill(5)}.dae" scale="${10*mesh_size} ${10*mesh_size} 1"/>
+        </geometry>
+      </visual>
+    </link>
+    <joint
+      name="apriltag_joint"
+      type="fixed">
+      <origin
+        xyz="0.0 0 0.059"
+        rpy="0 1.57 0" />
+      <parent link="${tf_prefix}laser" />
+      <child link="${namespace}${name}" />
+      <axis
+        xyz="0 0 0" />
+    </joint>
+    <!-- we use Gazebo material to put the texture onto the marker. Note mu1=mu2=0 for no friction. -->
+    <gazebo reference="${namespace}${name}">
+      <!-- <material>Gazebo/Red</material> -->
+      <turnGravityOff>false</turnGravityOff>
+      <selfCollide>false</selfCollide>
+      <mu1>0</mu1>
+      <mu2>0</mu2>
+      <kp>1000000.0</kp>
+      <kd>1.0</kd>
+    </gazebo>
+  </xacro:macro>
     <link name="${tf_prefix}base_link"/>
     <link name="${tf_prefix}chassis">
@@ -84,5 +126,5 @@
       <child link="${tf_prefix}chassis" />
     </joint>
-  <link name="${tf_prefix}chassis_inertia">
+    <link name="${tf_prefix}chassis_inertia">
     <inertial>
         <origin
@@ -367,35 +409,4 @@
       <child
         link="${tf_prefix}laser" />
-      <axis
-        xyz="0 0 0" />
-    </joint>
-    <link name="${namespace}${name}">
-      <inertial>
-        <mass value="0.001" />
-        <origin xyz="0 0 0" rpy="0 0 0" />
-        <inertia ixx="0.00001" ixy="0" ixz="0" iyy="0.00001" iyz="0" izz="0.00002" />
-      </inertial>
-      <collision>
-        <origin xyz="0 0 0" rpy="0 0 0" />
-        <geometry>
-          <box size="${mesh_size} ${mesh_size} 0.001" />
-        </geometry>
-      </collision>
-      <visual>
-        <origin xyz="0 0 0" rpy="0 0 0" />
-        <geometry>
-          <!-- use Python str to convert family name and to generate leading zeros -->
-          <mesh filename="package://tams_apriltags/meshes/tag${str(family).replace( 'h', '_' )}_${str(ID).zfill(5)}.dae" scale="${10*mesh_size} ${10*mesh_size} 1"/>
-        </geometry>
-      </visual>
-    </link>
-    <joint
-      name="apriltag_joint"
-      type="fixed">
-      <origin
-        xyz="0.0 0 0.059"
-        rpy="0 1.57 0" />
-      <parent link="${tf_prefix}laser" />
-      <child link="${namespace}${name}" />
       <axis
         xyz="0 0 0" />
@@ -434,5 +445,5 @@
       <minDepth>0.001</minDepth>
     </gazebo>
-  <!-- controller -->
+    <!-- controller -->
     <gazebo>
       <plugin name="differential_drive_controller"
@@ -460,19 +471,3 @@
       </plugin>
     </gazebo>
-    <!-- we use Gazebo material to put the texture onto the marker. Note mu1=mu2=0 for no friction. -->
-    <gazebo reference="${namespace}${name}">
-      <!-- <material>Gazebo/Red</material> -->
-      <turnGravityOff>false</turnGravityOff>
-      <selfCollide>false</selfCollide>
-      <mu1>0</mu1>
-      <mu2>0</mu2>
-      <kp>1000000.0</kp>
-      <kd>1.0</kd>
-    </gazebo>
-  <!--   <joint name="apriltag_joint" type="fixed">
-      <xacro:insert_block name="origin" />
-      <parent link="${tf_prefix}laser" />
-      <child link="${namespace}${name}" />
-    </joint>  -->
-  </xacro:macro>
 </robot>
